File: Electrical/Warmup Project/Electrical Diagrams/Circuit diagrams kicad/Updated Circuit Diagram/Updated Circuit Diagram.kicad_sch (KiCad schematic)
At the start: 30 parts, among them M1 Motor_DC, M2 Motor_DC, M3 Motor_DC, U3 MCP2562-H_SN, U4 Teensy4.1, U5 MCP2562-H_SN, U7 MCP2562-H_SN, U8 ADS1220IPWR

Commit message: Updated Code
Parts:
- removed AMT213D-V, AMT213D-V1, AMT213D-V2: (no value), symbol Rotary_encoder:Encoder
- removed E_STOP, E_STOP1: SW_Push_Open_Dual, symbol Switch:SW_Push_Open_Dual
- removed M1, M2: Motor_DC, symbol Motor:Motor_DC
- removed U1, U2, U6: (no value), symbol New_Library:O_Drive_Pro
- added E_STOP3, E_STOP4: SW_Push_Open_Dual, symbol Switch:SW_Push_Open_Dual
- added M4, M5: Motor_DC, symbol Motor:Motor_DC
Connections:
- net +24V: now also E_STOP3.1, E_STOP4.1
- net GNDPWR: now also M4.2 (-), M5.2 (-)
- net at M3.1 (+): now also R2.1, U7.7 (CANH)
- net at R2.2, U7.6 (CANL): now also E_STOP2.2
- net at R3.1, U3.7 (CANH): now also M4.1 (+)
- net at R3.2, U3.6 (CANL): now also E_STOP3.2
- net at R4.1, U5.7 (CANH): now also M5.1 (+)
- net at R4.2, U5.6 (CANL): now also E_STOP4.2
Other:
- note added: "CubeMars AK45-10"
- note removed: "Maxon 283858"
- note removed: "Maxon 539482"
- moved on the sheet: E_STOP2
